File: spool.kicad_pcb (KiCad board)
At the start: 4 copper layers, 80 x 87 mm, 116 parts, among them J1 USB_B_Micro, J10 Switch_1, J11 Switch_1, J12 Conn_02x10_Counter_Clockwise, J13 Conn_02x10_Counter_Clockwise, J2 SWD, J3 Switch_1, J4 Switch_1, J5 Switch_1, J6 Switch_2, J7 Conn_01x02, J8 Conn_01x08, J9 Conn_01x05, M1 Motor_DC, Q1 AO3400A, Q2 2N7002, SW1 USB_BOOT, SW2 RESET, SW3 SW_Push_DPDT, SW4 SW_Coded_SH-7010, SW5 SW_Push_DPDT, U1 TPS63070RNMR, U10 HT75xx-1-SOT89, U11 TPL0401B-10-Q1, U12 BS612, U14 PCF8563T, U2 RPI-441C1, U3 AS5600-ASOT, U4 RPI-441C1, U5 RPI-441C1, U6 DRV8871DDA, U7 W25Q128JVS, U8 RP2040, U9 BS612, Y1 Crystal_GND24, Y2 Crystal

Commit message: WIP
Parts:
- removed J10, J11: Switch_1, Connector_PinHeader_2.54mm:PinHeader_1x02_P2.54mm_Vertical
- removed J12: Conn_02x10_Counter_Clockwise, Connector_PinHeader_2.54mm:PinHeader_2x10_P2.54mm_Vertical
- removed J9: Conn_01x05, Connector_PinHeader_2.54mm:PinHeader_1x05_P2.54mm_Vertical
- removed R13: 1k, Resistor_SMD:R_0603_1608Metric
- added C33: 100n, Capacitor_SMD:C_0402_1005Metric, F.Cu at (-0.83, -33.1)
- added C34: 100uF, Capacitor_SMD:CP_Elec_6.3x7.7, F.Cu at (-7.12, -30.5)
- added C35: 100uF, Capacitor_SMD:CP_Elec_6.3x7.7, F.Cu at (-14.2, -30.5)
- added D10: D, Diode_SMD:D_SOD-323_HandSoldering, F.Cu at (9.62, -24.4)
- added D11: D, Diode_SMD:D_SOD-323_HandSoldering, F.Cu at (26.6, 42.6)
- added D4: D, Diode_SMD:D_SOD-323_HandSoldering, F.Cu at (7.58, -28.4)
- added D5: D, Diode_SMD:D_SOD-323_HandSoldering, F.Cu at (11.5, -28.5)
- added D6: D, Diode_SMD:D_SOD-323_HandSoldering, F.Cu at (10.4, 2.78)
- added D7: D, Diode_SMD:D_SOD-323_HandSoldering, F.Cu at (7.59, -24.4)
- added D8: D, Diode_SMD:D_SOD-323_HandSoldering, F.Cu at (5.68, -24.4)
- added D9: D, Diode_SMD:D_SOD-323_HandSoldering, F.Cu at (11.5, -24.4)
- added J14: Conn_01x07, Connector_PinHeader_2.54mm:PinHeader_1x07_P2.54mm_Vertical, F.Cu at (-29.4, 28.9)
- added R33: 47k, Resistor_SMD:R_0805_2012Metric_Pad1.20x1.40mm_HandSolder, F.Cu at (9.03, -31.9)
- BZ1: footprint cacophony-library:BUZ-TH_BD9.0-P5.00-D0.6-FD -> cacophony-library:BUZ-TH_BD9.0-P4.00-D0.6-FD
- H1, H2, H3, H4: footprint cacophony-library:MountingHole_3.2mm_M3 -> cacophony-library:MountingHole_3.5mm_M3
- J13: footprint Connector_PinHeader_2.54mm:PinHeader_2x10_P2.54mm_Vertical -> cacophony-library:test-headers
- L1: value INDUCTOR -> 1.5H
- R10, R12: value 1k -> 100k; footprint Resistor_SMD:R_0603_1608Metric -> Resistor_SMD:R_0402_1005Metric
- R11, R5, R8: value 1k -> 47Ω
- R15: value R -> 47k
- R6, R7, R9: value 1k -> 10k; footprint Resistor_SMD:R_0603_1608Metric -> Resistor_SMD:R_0402_1005Metric
- moved M1 62.0 mm to (-18.4, -37.9), turned to 180 degrees
- moved R15 57.5 mm to (3.25, -34.2), turned to 0 degrees
- moved U6 57.4 mm to (0.89, -29.9)
- moved R9 56.6 mm to (-27.7, 18.0), turned to 90 degrees
- moved R12 50.1 mm to (4.08, -25.1), turned to -90 degrees
- moved R10 43.2 mm to (13.6, -27.1), turned to 0 degrees
- moved Q1 34.4 mm to (13.4, 0.21), turned to 0 degrees
- moved R14 30.2 mm to (11.0, -0.25), turned to -90 degrees
- moved SW2 21.0 mm to (-20.5, 19.1)
- moved SW1 14.5 mm to (-2.70, 47.4), turned to 180 degrees
- moved J2 13.5 mm to (-21.3, 24.2), turned to 90 degrees
- moved SW4 11.7 mm to (19.0, 36.7)
- moved J8 11.5 mm to (-13.8, 41.2)
- moved R28 11.0 mm to (-5.77, -13.3), turned to 0 degrees
- moved BZ1 10.7 mm to (30.2, 48.1), turned to -90 degrees
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Connections:
- J13 pad 10: unconnected-(J13-Pin_10-Pad10) -> PIN_10
- J13 pad 12: unconnected-(J13-Pin_12-Pad12) -> PIN_12
- J13 pad 14: unconnected-(J13-Pin_14-Pad14) -> PIN_14
- J13 pad 16: unconnected-(J13-Pin_16-Pad16) -> PIN_16
- J13 pad 18: unconnected-(J13-Pin_18-Pad18) -> PIN_18
- J13 pad 2: unconnected-(J13-Pin_2-Pad2) -> PIN_2
- J13 pad 20: unconnected-(J13-Pin_20-Pad20) -> PIN_20
- J13 pad 4: unconnected-(J13-Pin_4-Pad4) -> PIN_4
- J13 pad 6: unconnected-(J13-Pin_6-Pad6) -> PIN_6
- J13 pad 8: unconnected-(J13-Pin_8-Pad8) -> PIN_8
- R10 pad 1: /PHOTO_2_OUT_PHY -> Net-(D10-K)
- R12 pad 1: /PHOTO_3_OUT_PHY -> Net-(D4-A)
- R12 pad 2: PHOTO_3_OUT -> GND
- R6 pad 1: /PHOTO_1_OUT_PHY -> +3V3
- R6 pad 2: PHOTO_1_OUT -> PHOTO_HOME_OUT
- R7 pad 1: /PHOTO_1_OUT_PHY -> +3V3
- R7 pad 2: GND -> PHOTO_RELEASE_OUT
- R9 pad 1: /PHOTO_2_OUT_PHY -> +3V3
- R9 pad 2: PHOTO_2_OUT -> PHOTO_RESET_OUT
- U2 pad 3: +3V3 -> PHOTO_HOME_OUT
- U2 pad 4: /PHOTO_1_OUT_PHY -> GND
- U4 pad 3: +3V3 -> PHOTO_RELEASE_OUT
- U4 pad 4: /PHOTO_2_OUT_PHY -> GND
- U5 pad 3: +3V3 -> PHOTO_RESET_OUT
- U5 pad 4: /PHOTO_3_OUT_PHY -> GND
- U6 pad 2: H_IN2 -> Net-(D4-A)
- U6 pad 3: H_IN1 -> Net-(D10-K)
- U8 pad 11: R_ENC_1 -> SWITCH_2
- U8 pad 12: GPIO_9 -> H_IN1
- U8 pad 13: GPIO_10 -> H_IN2
- U8 pad 14: GPIO_11 -> Net-(D6-A)
- U8 pad 17: PHOTO_2_OUT -> PHOTO_RELEASE_OUT
- U8 pad 18: PHOTO_1_OUT -> PHOTO_HOME_OUT
- U8 pad 29: EN_PHOTO -> PHOTO_RESET_OUT
- U8 pad 30: PHOTO_3_OUT -> GPIO_19
- U8 pad 31: H_IN1 -> GPIO_20
- U8 pad 32: H_IN2 -> GPIO_21
- U8 pad 36: RP2040_TX_IN -> RP2040_TX_OUT
- U8 pad 37: RP2040_RX_IN -> RP2040_RX_OUT
- U8 pad 40: RP2040_TX_OUT -> RP2040_TX_IN
- U8 pad 41: RP2040_RX_OUT -> RP2040_RX_IN
- U8 pad 5: SWITCH_1 -> R_ENC_4
- U8 pad 6: SWITCH_2 -> R_ENC_2
- U8 pad 7: R_ENC_2 -> R_ENC_1
- U8 pad 8: R_ENC_4 -> R_ENC_8
- U8 pad 9: R_ENC_8 -> SWITCH_1
Routing:
- net PHOTO_RESET_OUT: track 0.00 -> 89.0 mm, vias 0 -> 3
- net PHOTO_RELEASE_OUT: track 0.00 -> 87.0 mm, vias 0 -> 1
- net PHOTO_HOME_OUT: track 0.00 -> 53.3 mm
- net H_IN2: track 12.2 -> 62.7 mm, vias 0 -> 2
- net H_IN1: track 12.6 -> 62.4 mm, vias 0 -> 2
- net PHOTO_1_OUT: track 45.2 -> 0.00 mm
- net +12V: track 125.9 -> 162.0 mm, vias 0 -> 18
- net PHOTO_2_OUT: track 35.7 -> 0.00 mm
- net Net-(D6-A): track 0.00 -> 28.7 mm, vias 0 -> 2
- net +3V3_Lin: track 84.4 -> 58.2 mm, vias 4 -> 3
- net GPIO_9: track 24.5 -> 0.00 mm
- net Net-(M1--): track 6.76 -> 30.4 mm
- net PHOTO_3_OUT: track 23.5 -> 0.00 mm
- net GPIO_10: track 22.8 -> 0.00 mm
- net GPIO_11: track 22.5 -> 0.00 mm
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- added copper zone on In2.Cu, net +12V
Other:
- board size 80 x 87 mm -> 80 x 95 mm
- board text added: "12V"
- board text added: "3V3"
- board text added: "CCW"
- board text added: "CW"
- board text added: "Cacophony Spool Controller ${TAG}"
- board text added: "RX_IN"
- board text added: "RX_OUT"
- board text added: "TX_IN"
- board text added: "TX_OUT"
- board text removed: "CLK"
- board text removed: "SWD"
