File: spool.kicad_sch (KiCad schematic)
At the start: 116 parts, among them J1 USB_B_Micro, J10 Switch_1, J11 Switch_1, J12 Conn_02x10_Counter_Clockwise, J13 Conn_02x10_Counter_Clockwise, J2 SWD, J3 Switch_1, J4 Switch_1, J5 Switch_1, J6 Switch_2, J7 Conn_01x02, J8 Conn_01x08, J9 Conn_01x05, M1 Motor_DC, Q1 AO3400A, Q2 2N7002, SW1 USB_BOOT, SW2 RESET, SW3 SW_Push_DPDT, SW4 SW_Coded_SH-7010, SW5 SW_Push_DPDT, U1 TPS63070RNMR, U10 HT75xx-1-SOT89, U11 TPL0401B-10-Q1, U12 BS612, U14 PCF8563T, U2 RPI-441C1, U3 AS5600-ASOT, U4 RPI-441C1, U5 RPI-441C1, U6 DRV8871DDA, U7 W25Q128JVS, U8 RP2040, U9 BS612, Y1 Crystal_GND24, Y2 Crystal

Commit message: WIP
Parts:
- removed J10, J11: Switch_1, Connector_PinHeader_2.54mm:PinHeader_1x02_P2.54mm_Vertical, symbol Connector_Generic:Conn_01x02
- removed J12: Conn_02x10_Counter_Clockwise, Connector_PinHeader_2.54mm:PinHeader_2x10_P2.54mm_Vertical, symbol Connector_Generic:Conn_02x10_Counter_Clockwise
- removed J9: Conn_01x05, Connector_PinHeader_2.54mm:PinHeader_1x05_P2.54mm_Vertical, symbol Connector_Generic:Conn_01x05
- removed R13: 1k, Resistor_SMD:R_0603_1608Metric, symbol Device:R
- added C33: 100n, Capacitor_SMD:C_0402_1005Metric, symbol Device:C_Small
- added C34, C35: 100uF, Capacitor_SMD:CP_Elec_6.3x7.7, symbol Device:C_Polarized_Small_US
- added D10, D11, D4, D5, D6, D7, D8, D9: D, Diode_SMD:D_SOD-323_HandSoldering, symbol Device:D
- added J14: Conn_01x07, Connector_PinHeader_2.54mm:PinHeader_1x07_P2.54mm_Vertical, symbol Connector_Generic:Conn_01x07
- added R33: 47k, Resistor_SMD:R_0805_2012Metric_Pad1.20x1.40mm_HandSolder, symbol Device:R
- BZ1: footprint cacophony-library:BUZ-TH_BD9.0-P5.00-D0.6-FD -> cacophony-library:BUZ-TH_BD9.0-P4.00-D0.6-FD; LCSC C96102 -> C96256
- H1, H2, H3, H4: footprint cacophony-library:MountingHole_3.2mm_M3 -> cacophony-library:MountingHole_3.5mm_M3
- J13: footprint Connector_PinHeader_2.54mm:PinHeader_2x10_P2.54mm_Vertical -> cacophony-library:test-headers
- L1: value INDUCTOR -> 1.5H
- R10, R12: value 1k -> 100k; footprint Resistor_SMD:R_0603_1608Metric -> Resistor_SMD:R_0402_1005Metric; LCSC C21190 -> C25741
- R11, R5, R8: value 1k -> 47Ω; LCSC C21190 -> C23182
- R15: value R -> 47k
- R6, R7, R9: value 1k -> 10k; footprint Resistor_SMD:R_0603_1608Metric -> Resistor_SMD:R_0402_1005Metric; LCSC C21190 -> C25744
Connections:
- net GPIO_10 is gone; now on net H_IN2: U8.13 (GPIO10)
- net GPIO_9 is gone; now on net H_IN1: U8.12 (GPIO9)
- net +12V: now also C33.1, C34.1, C35.1
- net +3V3: now also R6.1, R7.1, R9.1, D11.1 (K), J14.2 (Pin_2); no longer U2.3, U4.3, U5.3
- net EN_PHOTO: now also D4.1 (K), D5.1 (K), D6.1 (K); no longer U8.29 (GPIO18)
- net GND: now also R12.2, U2.4, U4.4, U5.4, C33.2, C34.2, C35.2, J14.1 (Pin_1), R33.2; no longer R7.2
- net GPIO_27: now also J14.4 (Pin_4)
- net GPIO_34: now also J14.3 (Pin_3)
- net H_IN1: now also D9.2 (A); no longer U6.3 (IN1), U8.31 (GPIO20)
- net H_IN2: now also D8.2 (A); no longer U6.2 (IN2), U8.32 (GPIO21)
- net RP2040_RX_IN: now also U8.41 (GPIO29_ADC3); no longer U8.37 (GPIO25)
- net RP2040_RX_OUT: now also U8.37 (GPIO25); no longer U8.41 (GPIO29_ADC3)
- net RP2040_TX_IN: now also U8.40 (GPIO28_ADC2); no longer U8.36 (GPIO24)
- net RP2040_TX_OUT: now also U8.36 (GPIO24); no longer U8.40 (GPIO28_ADC2)
- net R_ENC_1: now also U8.7 (GPIO5); no longer U8.11 (GPIO8)
- net R_ENC_2: now also U8.6 (GPIO4); no longer U8.7 (GPIO5)
- net R_ENC_4: now also U8.5 (GPIO3); no longer U8.8 (GPIO6)
- net R_ENC_8: now also U8.8 (GPIO6); no longer U8.9 (GPIO7)
- net SWITCH_1: now also U8.9 (GPIO7); no longer U8.5 (GPIO3)
- net SWITCH_2: now also U8.11 (GPIO8); no longer U8.6 (GPIO4)
- net PIN_10: now reaches J13.10 (Pin_10)
- net PIN_12: now reaches J13.12 (Pin_12)
- net PIN_14: now reaches J13.14 (Pin_14)
- net PIN_16: now reaches J13.16 (Pin_16)
- net PIN_18: now reaches J13.18 (Pin_18)
- net PIN_2: now reaches J13.2 (Pin_2)
- net PIN_20: now reaches J13.20 (Pin_20)
- net PIN_4: now reaches J13.4 (Pin_4)
- net PIN_6: now reaches J13.6 (Pin_6)
- net PIN_8: now reaches J13.8 (Pin_8)
- net at BZ1.2 (-), R31.1: now also D11.2 (A)
- net at R15.1, U6.4 (ILIM): now also R33.1
- net GPIO_11: no longer names the net of U8.14 (GPIO11)
- net GPIO_11: now also D6.2 (A)
- net PHOTO_1_OUT renamed PHOTO_HOME_OUT
- net PHOTO_HOME_OUT: now also U2.3
- removed net PHOTO_1_OUT_PHY: R6.1, R7.1, U2.4
- net PHOTO_2_OUT renamed PHOTO_RELEASE_OUT
- net PHOTO_RELEASE_OUT: now also R7.2, U4.3, D10.2 (A); no longer R9.2
- removed net PHOTO_2_OUT_PHY: R10.1, R9.1, U4.4
- net PHOTO_3_OUT renamed GPIO_19
- net GPIO_19: now also J14.5 (Pin_5); no longer R12.2
- net PHOTO_3_OUT_PHY: no longer names the net of R12.1
- net PHOTO_3_OUT_PHY: now also U6.2 (IN2), D4.2 (A), D7.1 (K), D8.1 (K); no longer U5.4
- new net: D10.1 (K), D5.2 (A), D9.1 (K), R10.1, U6.3 (IN1)
- new net GPIO_20: J14.6 (Pin_6), U8.31 (GPIO20)
- new net GPIO_21: J14.7 (Pin_7), U8.32 (GPIO21)
- new net PHOTO_RESET_OUT: D7.2 (A), R9.2, U5.3, U8.29 (GPIO18)
- no-connect marks 45 -> 15
Other:
- note added: "Breakout pins"
- note added: "Buzzer & LED Status indicators"
- note added: "Generic plugs for in/out digital signals"
- note added: "I2C bus pullups"
- note added: "Linear power supply"
- note added: "MS621FE"
- note added: "Magnet rotarty position sensor"
- note added: "Make sure C21 is close to pin 44 of RP2040"
- note added: "Motor driver"
- note added: "Mounting holes"
- note added: "Night/Day Mode Select"
- note added: "PIRs"
- note added: "Photo Interrupter Sensors"
- note added: "Power"
- note added: "Power/Data plug"
- note added: "Program Select Switch"
- note added: "RP2040"
- note added: "RTC"
- note added: "Sensitivity for PIRs"
- note added: "Switching power supply"
- note removed: "Cage switch"
- note removed: "Make sure C10 is close to pin 44 of RP2040"
- note removed: "Night/Day mode select"
- note removed: "Program Select"
- moved on the sheet: BT1, BZ1, C1, C10, C11, C12, C13, C14, C15, C16, C17, C18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

Commit message: Add changes for magnet release
Parts:
- removed R11, R5, R8: 47Ω, Resistor_SMD:R_0603_1608Metric, symbol Device:R
- removed R9: 10k, Resistor_SMD:R_0402_1005Metric, symbol Device:R
- removed U2, U4, U5: RPI-441C1, cacophony-library:OPTO-TH_RPI-441C1, symbol cacophony-library:RPI-441C1
- added C101, C102, C104: 100n, Capacitor_SMD:C_0402_1005Metric, symbol Device:C_Small
- added C103, C105: 2.2uF, Capacitor_SMD:C_0402_1005Metric, symbol Device:C_Small
- added D101: D, Diode_SMD:D_SOD-323_HandSoldering, symbol Device:D
- added L101: ElectromagneticActor, Connector_JST:JST_XA_B02B-XASK-1-A_1x02_P2.50mm_Vertical, symbol Device:ElectromagneticActor
- added Q101: Q_NMOS_GSD, Package_TO_SOT_SMD:SOT-23, symbol Transistor_FET:Q_NMOS_GSD
- added R101, R102: 100k, Resistor_SMD:R_0402_1005Metric, symbol Device:R
- added R103: R_Shunt, cacophony-library:R_1206_Shunt, symbol Device:R_Shunt
- added R104, R105: 150Ω, Resistor_SMD:R_0603_1608Metric, symbol Device:R
- added TP101: TestPoint, cacophony-library:TP_PAD, symbol cacophony-library:TestPoint
- added U101: MMA8451QR1, cacophony-library:QFN-16_L3.0-W3.0-P0.50-TL_FXOS8700CQR1, symbol cacophony-library:MMA8451QR1
- added U102: INA219AxDCN, Package_TO_SOT_SMD:SOT-23-8, symbol Sensor_Energy:INA219AxDCN
- added U103, U104: DY-ITR8402, cacophony-library:OPTO-TH_DY-ITR8402, symbol cacophony-library:DY-ITR8402
- R33: value 47k -> 33k; LCSC C17713 -> C17633
- U7: footprint Package_SO:SOIC-8_5.23x5.23mm_P1.27mm -> Package_SO:SOIC-8_5.3x5.3mm_P1.27mm
- U8: LCSC Part (none) -> C2040
Connections:
- net PIN_6 is gone; now on net SDA: J13.6 (Pin_6)
- net PIN_8 is gone; now on net SCL: J13.8 (Pin_8)
- net +12V: now also D101.1 (K), L101.1 (-), R103.4; no longer C33.1, C34.1, C35.1, U6.5 (VM)
- net +3V3: now also C101.1, C103.1, C104.1, C105.1, R104.1, R105.1, U101.1 (VDDIO), U101.14 (VDD), U102.4 (VS)
- net GND: now also C101.2, C102.2, C103.2, C104.2, C105.2, Q101.2 (S), R101.2, R102.2, U101.10 (GND), U101.12 (GND), U101.5 (GND), U101.7 (SA0), U102.3 (GND), U103.4, U104.4
- net PHOTO_1_ANODE: now also R104.2, U104.1
- net PHOTO_2_ANODE: now also R105.2, U103.1
- net PHOTO_CATHODE: now also U103.2, U104.2
- net PHOTO_HOME_OUT: now also D10.2 (A), U104.3
- net PHOTO_RESET_OUT: now also R7.2, U8.17 (GPIO14), U103.3; no longer U8.29 (GPIO18)
- net R_ENC_1: now also U8.6 (GPIO4); no longer U8.7 (GPIO5)
- net R_ENC_2: now also U8.7 (GPIO5); no longer U8.6 (GPIO4)
- net SCL: now also U101.4 (SCL), U102.5 (SCL)
- net SDA: now also U101.6 (SDA), U102.6 (SDA)
- net GPIO_19: no longer names the net of J14.5 (Pin_5)
- net GPIO_19: no longer U8.30 (GPIO19)
- removed net PHOTO_RELEASE_OUT: D10.2 (A), R7.2, U8.17 (GPIO14)
- net PIN_10: no longer names the net of J13.10 (Pin_10)
- net PIN_12: no longer names the net of J13.12 (Pin_12)
- net PIN_14: no longer names the net of J13.14 (Pin_14)
- net PIN_16: no longer names the net of J13.16 (Pin_16)
- net PIN_18: no longer names the net of J13.18 (Pin_18)
- net PIN_2: no longer names the net of J13.2 (Pin_2)
- net PIN_20: no longer names the net of J13.20 (Pin_20)
- net PIN_4: no longer names the net of J13.4 (Pin_4)
- new net: R101.1, U102.7 (A0)
- new net: R102.1, U102.8 (A1)
- new net: TP101.1, U101.9 (INT2)
- new net: R103.2, U102.2 (IN-)
- new net: R103.3, U102.1 (IN+)
- new net: C102.1, U101.2 (BYP)
- new net: D101.2 (A), L101.2 (+), Q101.3 (D)
- new net Accel INT1: U101.11 (INT1), U8.30 (GPIO19)
- new net RELEASE: Q101.1 (G), U8.29 (GPIO18)
- new net h_bridge_vcc: C33.1, C34.1, C35.1, R103.1, U6.5 (VM)
- no-connect marks 15 -> 29
Other:
- note added: "Accelerometer"
- note added: "Magnet Release"
- moved on the sheet: C33, C34, C35, D10, D4, D5, D7, D8, D9, M1, R10, R12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
