File: spool/spool.kicad_pcb (KiCad board)
At the start: 4 copper layers, 80 x 95 mm, 124 parts, among them J1 USB_B_Micro, J13 Conn_02x10_Counter_Clockwise, J14 Conn_01x07, J2 SWD, J3 Switch_1, J4 Switch_1, J5 Switch_1, J6 Switch_2, J7 Conn_01x02, J8 Conn_01x08, M1 Motor_DC, Q1 AO3400A, Q2 2N7002, SW1 USB_BOOT, SW2 RESET, SW3 SW_Push_DPDT, SW4 SW_Coded_SH-7010, SW5 SW_Push_DPDT, U1 TPS63070RNMR, U10 HT75xx-1-SOT89, U11 TPL0401B-10-Q1, U12 BS612, U14 PCF8563T, U2 RPI-441C1, U3 AS5600-ASOT, U4 RPI-441C1, U5 RPI-441C1, U6 DRV8871DDA, U7 W25Q128JVS, U8 RP2040, U9 BS612, Y1 Crystal_GND24, Y2 Crystal

Commit message: WIP
Parts:
- added C36: 22uF, Capacitor_SMD:C_0805_2012Metric, F.Cu at (-29.8, 3.88)
- added C37: 22uF, Capacitor_SMD:C_0805_2012Metric, F.Cu at (-31.8, 3.88)
- C34, C35: value 100uF -> 470uF; footprint Capacitor_SMD:CP_Elec_6.3x7.7 -> Capacitor_SMD:CP_Elec_8x10.5
- moved C35 42.3 mm to (28.0, -28.0), turned to 180 degrees
- moved M1 39.1 mm to (20.7, -37.6)
- moved C34 37.6 mm to (28.0, -17.0), turned to 180 degrees
- moved J13 35.5 mm to (-15.9, -23.3), turned to 90 degrees
- moved C33 23.0 mm to (22.0, -30.7), turned to -90 degrees
- moved U6 17.7 mm to (18.5, -29.1), turned to 90 degrees
- moved R15 13.5 mm to (12.7, -24.5), turned to 90 degrees
- moved R12 10.5 mm to (13.4, -20.2), turned to 180 degrees
- moved D4 10.3 mm to (15.3, -21.6)
- moved D10 10.3 mm to (17.4, -17.6)
- moved D7 10.3 mm to (15.3, -17.6)
- moved D8 10.3 mm to (13.4, -17.6)
- moved D9 10.3 mm to (19.3, -17.6)
- moved R10 8.96 mm to (19.3, -20.2)
- moved D5 8.93 mm to (17.2, -21.6)
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Connections:
- D10 pad 2: PHOTO_RELEASE_OUT -> PHOTO_RESET_OUT
- D7 pad 2: PHOTO_RESET_OUT -> PHOTO_RELEASE_OUT
- J13 pad 10: PIN_10 -> unconnected-(J13-Pin_10-Pad10)
- J13 pad 11: GND -> +3V3
- J13 pad 12: PIN_12 -> unconnected-(J13-Pin_12-Pad12)_2
- J13 pad 13: GND -> +3V3
- J13 pad 14: PIN_14 -> unconnected-(J13-Pin_14-Pad14)_2
- J13 pad 15: GND -> +3V3
- J13 pad 16: PIN_16 -> unconnected-(J13-Pin_16-Pad16)
- J13 pad 18: PIN_18 -> unconnected-(J13-Pin_18-Pad18)_2
- J13 pad 2: PIN_2 -> unconnected-(J13-Pin_2-Pad2)
- J13 pad 20: PIN_20 -> unconnected-(J13-Pin_20-Pad20)_1
- J13 pad 4: PIN_4 -> unconnected-(J13-Pin_4-Pad4)
- J13 pad 5: +3V3 -> +12V
- J13 pad 6: PIN_6 -> unconnected-(J13-Pin_6-Pad6)_2
- J13 pad 7: +3V3 -> +12V
- J13 pad 8: PIN_8 -> unconnected-(J13-Pin_8-Pad8)
Routing:
- net +12V: track 162.0 -> 200.7 mm, vias 18 -> 16
- net GND: track 55.5 -> 80.0 mm, vias 82 -> 76
- net Net-(M1--): track 30.4 -> 6.28 mm
- net Net-(M1-+): track 21.8 -> 6.26 mm
- net PHOTO_RELEASE_OUT: track 87.0 -> 74.7 mm
- net EN_PHOTO: track 41.3 -> 31.0 mm
- net H_IN2: track 62.7 -> 52.7 mm
- net +3V3: track 43.9 -> 51.5 mm
- net PHOTO_RESET_OUT: track 89.0 -> 94.8 mm
- net H_IN1: track 62.4 -> 56.6 mm
- net Net-(U6-ILIM): track 6.77 -> 11.9 mm, vias 0 -> 1
- net PIN_8: track 5.08 -> 0.00 mm
- net PIN_6: track 5.08 -> 0.00 mm
- net PIN_4: track 5.08 -> 0.00 mm
- net PIN_20: track 5.08 -> 0.00 mm
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