File: spool/spool.kicad_pcb (KiCad board)
At the start: 4 copper layers, 80 x 99 mm, 157 parts, among them J1 USB_B_Micro, J13 Conn_02x10_Counter_Clockwise, J1901 TC2030, J2 SWD, J3 Conn_01x03, J4 Switch_1, J5 Conn_01x03, J6 Switch_2, J7 Conn_01x02, J8 Conn_01x08, J9 Switch_2, M1 Motor_DC, M2 Servo, M3 Servo, Q1 AO3400A, Q101 Q_NMOS_GSD, Q2 2N7002, SW1 USB_BOOT, SW2 RESET, SW4 SW_Coded_SH-7010, SW5 SW_Push_DPDT, U1 TPS63070RNMR, U10 HT75xx-1-SOT89, U102 INA219AxDCN, U103 DY-ITR8402, U104 DY-ITR8402, U106 M24C02-WMN, U14 PCF8563T, U2 PA_PIR, U3 AS5600-ASOT, U6 DRV8871DDA, U7 W25Q128JVS, U8 RP2040, U9 LMR14050S, Y1 Crystal_GND24, Y2 Crystal

Commit message: Added kicad-library as submodule and simplify schematic
Parts:
- removed D3: D, Diode_SMD:D_SOD-523
- removed J7: Conn_01x02, Connector_PinHeader_2.00mm:PinHeader_1x02_P2.00mm_Vertical
- removed JP1: SolderJumper_2_Bridged, Jumper:SolderJumper-2_P1.3mm_Bridged_RoundedPad1.0x1.5mm
- removed R42: 1k, Resistor_SMD:R_1206_3216Metric
- added R45: 1k, Resistor_SMD:R_0402_1005Metric, F.Cu at (-26.5, -25.0)
- added R46: 1k, Resistor_SMD:R_0402_1005Metric, F.Cu at (-26.5, -24.1)
- added R47: 1k, Resistor_SMD:R_0402_1005Metric, F.Cu at (-24.6, -25.0)
- added R48: 1k, Resistor_SMD:R_0402_1005Metric, F.Cu at (-24.6, -24.1)
- C1, C2, C28, C29: value 22uF -> 22uF 25V
- C104, C11, C12, C13, C14, C15, C16, C17, C18, C19, C22, C33, C39, C40: value 100n -> 100nF
- D10, D101, D11, D4, D5, D6, D7, D8, D9: footprint Diode_SMD:D_SOD-323_HandSoldering -> Diode_SMD:D_SOD-323
- D2: footprint Diode_SMD:D_SOD-123F -> Diode_SMD:D_SOD-323
- moved C10 3.76 mm to (0.13, -7.76), turned to 0 degrees
- moved R32 2.69 mm to (-19.6, 10.1), turned to -90 degrees
- moved J13 0.30 mm to (-18.0, 2.86)
- moved C30 0.14 mm to (-17.8, 7.92)
Connections:
- BT1 pad 1: Net-(BT1-+) -> /RTC_BAT
- TP2 pad 1: /RTC_BAT_SENSE -> /RTC_BAT
Routing:
- net /RTC_BAT: track 7.47 -> 22.8 mm
- net Net-(BT1-+): track 15.2 -> 0.00 mm
- net +3V3: track 69.4 -> 73.1 mm
- net Net-(R45-Pad2): track 0.00 -> 3.56 mm
- net /RTC_BAT_SENSE: track 3.25 -> 0.00 mm
- net /RTC_V_{DD}: track 7.96 -> 9.21 mm
- net /EX_PIR_POWER: track 2.44 -> 3.38 mm
- net +12V: track 19.7 -> 20.6 mm
- added copper zone on B.Cu, net GND
