File: spool/spool.kicad_pcb (KiCad board)
At the start: 4 copper layers, 80 x 99 mm, 157 parts, among them J1 USB_B_Micro, J13 Conn_02x10_Counter_Clockwise, J1901 TC2030, J2 SWD, J3 Conn_01x03, J4 Switch_1, J5 Conn_01x03, J6 Switch_2, J8 Conn_01x08, J9 Switch_2, M1 Motor_DC, M2 Servo, M3 Servo, Q1 AO3400A, Q101 Q_NMOS_GSD, Q2 2N7002, SW1 USB_BOOT, SW2 RESET, SW4 SW_Coded_SH-7010, SW5 SW_Push_DPDT, U1 TPS63070RNMR, U10 HT75xx-1-SOT89, U102 INA219AxDCN, U103 DY-ITR8402, U104 DY-ITR8402, U106 M24C02-WMN, U14 PCF8563T, U2 PA_PIR, U3 AS5600-ASOT, U6 DRV8871DDA, U7 W25Q128JVS, U8 RP2040, U9 LMR14050S, Y1 Crystal_GND24, Y2 Crystal

Commit message: Fix pin label
Other:
- board text added: "GPIO23"
- board text added: "Home"
- board text added: "Reset"
- board text removed: "GPIO12"
Changed lines of the file:
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@@
 		(layer "User.2")
 	)
-	(gr_text "GPIO12"
+	(gr_text "GPIO23"
 		(at -34.47 2.03 0)
 		(layer "F.SilkS")
@@
 		)
 	)
+	(gr_text "Home"
+		(at 16.99 0.32 0)
+		(layer "F.SilkS")
+		(effects
+			(font
+				(size 0.8128 0.8128)
+				(thickness 0.1524)
+				(bold yes)
+			)
+			(justify left bottom)
+		)
+	)
 	(gr_text "12V"
 		(at -29.38 38.95 90)
@@
 		(layer "F.SilkS")
 		(effects
+			(font
+				(size 0.8128 0.8128)
+				(thickness 0.1524)
+				(bold yes)
+			)
+			(justify left bottom)
+		)
+	)
+	(gr_text "Reset"
+		(at 15.75 5.95 340)
+		(layer "F.SilkS")
+		(effects

Commit message: Adding STM32 version
Parts:
- removed C11, C12, C13, C14, C15, C16, C17, C18, C19: 100nF, Capacitor_SMD:C_0402_1005Metric
- removed C20, C21: 1uF, Capacitor_SMD:C_0402_1005Metric
- removed J4: Switch_1, Connector_JST:JST_SH_BM02B-SRSS-TB_1x02-1MP_P1.00mm_Vertical
- removed J5: Conn_01x03, Connector_PinHeader_2.54mm:PinHeader_1x03_P2.54mm_Vertical
- removed J6: Switch_2, Connector_JST:JST_SH_BM02B-SRSS-TB_1x02-1MP_P1.00mm_Vertical
- removed J8: Conn_01x08, Connector_JST:JST_XA_S08B-XASK-1_1x08_P2.50mm_Horizontal
- removed M2, M3: Servo, Connector_JST:JST_XA_B03B-XASK-1-A_1x03_P2.50mm_Vertical
- removed R16, R17: 33ohm, Resistor_SMD:R_0402_1005Metric
- removed R18: DNF, Resistor_SMD:R_0402_1005Metric
- removed R43: 1k, Resistor_SMD:R_0402_1005Metric
- removed U7: W25Q128JVS, Package_SO:SOIC-8_5.3x5.3mm_P1.27mm
- removed Y1: Crystal_GND24, Crystal:Crystal_SMD_3225-4Pin_3.2x2.5mm
- added C41: 100nF, Capacitor_SMD:C_0402_1005Metric, F.Cu at (4.07, 36.5)
- added C42: 100nF, Capacitor_SMD:C_0402_1005Metric, F.Cu at (8.33, 29.5)
- added C43: 100nF, Capacitor_SMD:C_0402_1005Metric, F.Cu at (4.14, 39.5)
- added C44: 100nF, Capacitor_SMD:C_0402_1005Metric, F.Cu at (17.4, 44.4)
- added C45: 100nF, Capacitor_SMD:C_0402_1005Metric, F.Cu at (4.26, 43.7)
- added C51: 100nF, Capacitor_SMD:C_0402_1005Metric, F.Cu at (-3.51, 52.7)
- added D204: D_Zener, Diode_SMD:D_SOD-123, F.Cu at (-13.6, 53.0)
- added H14: MountingHole, cacophony-library:MountingHole_3.5mm_M3, F.Cu at (-21.4, 49.5)
- added H16: KeyHole, cacophony-library:3.0mm_key_hole, F.Cu at (-19.4, 37.5)
- added H17: KeyHole, cacophony-library:3.0mm_key_hole, F.Cu at (-10.5, 49.0)
- added J14: Conn_02x10_Counter_Clockwise, Connector_PinSocket_2.54mm:PinSocket_2x10_P2.54mm_Vertical, B.Cu at (-27.4, 43.5)
- added R201: 3.3M, Resistor_SMD:R_0603_1608Metric, F.Cu at (-9.60, 52.4)
- added R202: 1M, Resistor_SMD:R_0603_1608Metric, F.Cu at (-9.59, 53.9)
- added R24: 10k, Resistor_SMD:R_0402_1005Metric, F.Cu at (-6.56, -12.9)
- added R28: 10k, Resistor_SMD:R_0402_1005Metric, F.Cu at (-9.17, -13.6)
- added R36: 1k, Resistor_SMD:R_0402_1005Metric, F.Cu at (20.8, 36.8)
- added R49: 1k, Resistor_SMD:R_0402_1005Metric, F.Cu at (0.52, 41.8)
- added R5: 10k, Resistor_SMD:R_0402_1005Metric, F.Cu at (3.94, 31.1)
- added R50: 1k, Resistor_SMD:R_0402_1005Metric, F.Cu at (0.64, 43.0)
- added U5: MCP6001-OT, Package_TO_SOT_SMD:SOT-23-5, F.Cu at (-6.05, 53.1)
- C23, C24: value 12pF -> 100nF
- H11, H12, H13, H5, H6, H7, H8: value MountingHole -> KeyHole
- J1: value USB_B_Micro -> Conn_01x04; footprint cacophony-library:MICRO-USB-TH_MICRO-USB-A14 -> Connector_PinHeader_2.54mm:PinHeader_1x04_P2.54mm_Vertical
- J3: value Conn_01x03 -> Conn_01x04; footprint Connector_JST:JST_SH_BM03B-SRSS-TB_1x03-1MP_P1.00mm_Vertical -> Connector_PinHeader_2.54mm:PinHeader_1x04_P2.54mm_Vertical
- SW1: value USB_BOOT -> BOOT0
- U8: value RP2040 -> STM32L073RZTx; footprint cacophony-library:RP2040-QFN-56 -> Package_QFP:LQFP-64_10x10mm_P0.5mm
- moved J3 80.4 mm to (32.6, 23.4), turned to 0 degrees
- moved R35 74.8 mm to (0.63, 47.4), turned to 180 degrees
- moved R34 74.3 mm to (0.63, 46.4)
- moved R41 70.3 mm to (-0.62, 38.2)
- moved R45 65.9 mm to (-9.57, 38.7), turned to 180 degrees
- moved R47 65.1 mm to (-11.4, 38.7), turned to 180 degrees
- moved R46 64.1 mm to (-9.57, 37.8), turned to 180 degrees
- moved R23 63.6 mm to (-32.6, 25.0), turned to 90 degrees
- moved R48 63.2 mm to (-11.4, 37.8), turned to 180 degrees
- moved L2 62.7 mm to (-29.4, 34.6), turned to -90 degrees
- moved C37 62.3 mm to (-31.7, 24.9), turned to -90 degrees
- moved R26 61.9 mm to (-31.6, 23.3), turned to 180 degrees
- moved R27 61.8 mm to (-31.6, 21.8), turned to 0 degrees
- moved C50 58.1 mm to (-24.4, 38.1), turned to 0 degrees
- moved J9 57.7 mm to (7.70, -30.6), turned to 0 degrees
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Connections:
- C23 pad 1: GND -> +3V3
- C23 pad 2: Net-(U8-XIN) -> GND
- C24 pad 1: GND -> +3V3
- C24 pad 2: Net-(U8-XOUT) -> GND
- D6 pad 2: /EN_PHOTO_PHY -> Net-(D6-A)
- J1 pad 1: unconnected-(J1-VBUS-Pad1) -> /PB12
- J1 pad 2: /USB_D- -> /PB13
- J1 pad 3: /USB_D+ -> /PB14
- J1 pad 4: unconnected-(J1-ID-Pad4) -> /PB15
- J13 pad 4: GPIO_12 -> unconnected-(J13-Pin_4-Pad4)_1
- J3 pad 1: /EX_PIR_POWER -> /PC9
- J3 pad 2: GND -> /PC8
- J3 pad 3: PIR_EX -> /PC7
- R19 pad 1: /QSPI_SS -> /BOOT0
- R34 pad 1: /SERVO_2_PHY -> SERVO_SIG_2
- R34 pad 2: SERVO_2 -> /SERVO_2_PHY
- R35 pad 2: SERVO_1 -> SERVO_SIG_1
- R44 pad 1: /RP2040_TX_IN_PHY -> /TX_PHY
- R44 pad 2: RP2040_TX_IN -> TX_STM32
- R45 pad 1: /EX_PIR_POWER -> EX_PIR_POWER
- R46 pad 1: /EX_PIR_POWER -> EX_PIR_POWER
- SW1 pad 1: GND -> +3V3
- U8 pad 10: +3V3 -> unconnected-(U8-PC2-Pad10)
- U8 pad 11: R_ENC_1 -> unconnected-(U8-PC3-Pad11)
- U8 pad 12: /EN_PHOTO_PHY -> GND
- U8 pad 13: PHOTO_HOME_OUT -> +3V3
- U8 pad 14: PHOTO_RESET_OUT -> /APIR_PHY
- U8 pad 15: H_IN1 -> /PIR_EX_PHY
- U8 pad 16: H_IN2 -> /TX_PHY
- U8 pad 17: SDA -> /RX_PHY
- U8 pad 18: SCL -> GND
- U8 pad 19: GND -> +3V3
- U8 pad 2: NIGHT_ONLY -> unconnected-(U8-PC13-Pad2)
- U8 pad 20: Net-(U8-XIN) -> /BAT_DIV_PHY
- U8 pad 21: Net-(U8-XOUT) -> /SW_1_PHY
- U8 pad 22: +3V3 -> /SERVO_2_PHY
- U8 pad 23: +1V1 -> /SERVO_1_PHY
- U8 pad 24: /SWCLK -> /SW_2_PHY
- U8 pad 25: /SWD -> R_ENC_1
- U8 pad 26: /RUN -> R_ENC_4
- U8 pad 27: /RP2040_TX_IN_PHY -> R_ENC_2
- U8 pad 28: RP2040_RX_IN -> R_ENC_8
- U8 pad 29: EN_6V -> NIGHT_ONLY
- U8 pad 3: BUZZER -> unconnected-(U8-PC14-Pad3)
- U8 pad 30: /SERVO_1_PHY -> BUZZER
- U8 pad 31: /SERVO_2_PHY -> GND
- U8 pad 32: RELEASE -> +3V3
- U8 pad 33: +3V3 -> /PB12
- U8 pad 34: /PIR_EX_PHY -> /PB13
- U8 pad 35: GPIO_12 -> /PB14
- U8 pad 36: /RP2040_TX_OUT_PHY -> /PB15
- U8 pad 37: RP2040_RX_OUT -> /PC6
- U8 pad 38: /APIR_PHY -> /PC7
- U8 pad 39: /ADC1 -> /PC8
- U8 pad 4: /SW_1_PHY -> unconnected-(U8-PC15-Pad4)
- U8 pad 40: /ADC2 -> /PC9
- U8 pad 41: /ADC3 -> /EN_PHOTO_PHY
- U8 pad 42: +3V3 -> /USART_1_TX
- U8 pad 43: +3V3 -> /USART_1_RX
- U8 pad 44: +3V3 -> /USB_PHY_D-
- U8 pad 45: +1V1 -> /USB_PHY_D+
- U8 pad 46: /USB_PHY_D- -> /SWD
- U8 pad 47: /USB_PHY_D+ -> GND
- U8 pad 49: +3V3 -> /SWCLK
- U8 pad 5: R_ENC_2 -> unconnected-(U8-PH0-Pad5)
- U8 pad 50: +1V1 -> unconnected-(U8-PA15-Pad50)
- U8 pad 51: /QSPI_SD3 -> PHOTO_HOME_OUT
- U8 pad 52: /QSPI_SCLK -> PHOTO_RESET_OUT
- U8 pad 53: /QSPI_SD0 -> H_IN1
- U8 pad 54: /QSPI_SD2 -> H_IN2
- U8 pad 55: /QSPI_SD1 -> /SPOOL_REED_PHY
- U8 pad 56: /QSPI_SS -> RELEASE
- U8 pad 57: GND -> unconnected-(U8-PB5-Pad57)
- U8 pad 6: R_ENC_8 -> unconnected-(U8-PH1-Pad6)
- U8 pad 7: /SW_2_PHY -> /RUN
- U8 pad 8: /SPOOL_REED_PHY -> unconnected-(U8-PC0-Pad8)
- U8 pad 9: R_ENC_4 -> unconnected-(U8-PC1-Pad9)
Routing:
- net /PIR_EX_PHY: track 85.4 -> 7.48 mm, vias 2 -> 0
- net /SERVO_1_PHY: track 88.9 -> 13.0 mm, vias 2 -> 0
- net /SERVO_2_PHY: track 76.1 -> 12.0 mm, vias 2 -> 0
- net +3V3: track 73.1 -> 133.9 mm, vias 29 -> 28
- net GPIO_12: track 54.9 -> 0.00 mm, vias 1 -> 0
- net EN_6V: track 73.5 -> 39.4 mm, vias 2 -> 0
- net /SPOOL_REED_PHY: track 30.1 -> 60.2 mm
- net /EN_PHOTO_PHY: track 32.6 -> 2.57 mm
- net RP2040_RX_OUT: track 24.5 -> 0.00 mm
- net SERVO_SIG_2: track 0.00 -> 23.0 mm
- net /PC9: track 0.00 -> 22.6 mm
- net +6V: track 39.9 -> 17.8 mm
- net SERVO_SIG_1: track 0.00 -> 21.4 mm
- net Net-(D6-A): track 0.00 -> 21.1 mm
- net /PC8: track 0.00 -> 20.7 mm
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- removed copper zone on F.Cu, net +1V1
Other:
- board text added: "24H"
- board text added: "BOOT"
- board text added: "RUN"
- board text removed: "12V"
- board text removed: "3.3V"
- board text removed: "A1"
- board text removed: "A2"
- board text removed: "A3"
- board text removed: "BOOT MODE"
- board text removed: "GND"
- board text removed: "GPIO23"
- board text removed: "Night And Day"
- board text removed: "PIR_EX"
- board text removed: "RESET"
- board text removed: "RX_IN"
- board text removed: "RX_OUT"
- board text removed: "SCL"
- board text removed: "SDA"
- board text removed: "SW_1"
- board text removed: "SW_2"
- board text removed: "TX_IN"
- board text removed: "TX_OUT"
