File: spool/spool.kicad_sch (KiCad schematic)
At the start: 124 parts, among them J1 USB_B_Micro, J13 Conn_02x10_Counter_Clockwise, J14 Conn_01x07, J2 SWD, J3 Switch_1, J4 Switch_1, J5 Switch_1, J6 Switch_2, J7 Conn_01x02, J8 Conn_01x08, M1 Motor_DC, Q1 AO3400A, Q2 2N7002, SW1 USB_BOOT, SW2 RESET, SW3 SW_Push_DPDT, SW4 SW_Coded_SH-7010, SW5 SW_Push_DPDT, U1 TPS63070RNMR, U10 HT75xx-1-SOT89, U11 TPL0401B-10-Q1, U12 BS612, U14 PCF8563T, U2 RPI-441C1, U3 AS5600-ASOT, U4 RPI-441C1, U5 RPI-441C1, U6 DRV8871DDA, U7 W25Q128JVS, U8 RP2040, U9 BS612, Y1 Crystal_GND24, Y2 Crystal

Commit message: WIP
Parts:
- added C36, C37: 22uF, Capacitor_SMD:C_0805_2012Metric, symbol Device:C_Small
- C34, C35: value 100uF -> 470uF; footprint Capacitor_SMD:CP_Elec_6.3x7.7 -> Capacitor_SMD:CP_Elec_8x10.5; LCSC C3338 -> C178591
- R3: LCSC C723770 -> C852538
Connections:
- net +12V: now also J13.5 (Pin_5), J13.7 (Pin_7), C36.1, C37.1
- net +3V3: now also J13.11 (Pin_11), J13.13 (Pin_13), J13.15 (Pin_15); no longer J13.5 (Pin_5), J13.7 (Pin_7)
- net GND: now also C36.2, C37.2; no longer J13.11 (Pin_11), J13.13 (Pin_13), J13.15 (Pin_15)
- net PHOTO_RELEASE_OUT: now also D7.2 (A); no longer D10.2 (A)
- net PHOTO_RESET_OUT: now also D10.2 (A); no longer D7.2 (A)
- net PIN_10: no longer names the net of J13.10 (Pin_10)
- net PIN_12: no longer names the net of J13.12 (Pin_12)
- net PIN_14: no longer names the net of J13.14 (Pin_14)
- net PIN_16: no longer names the net of J13.16 (Pin_16)
- net PIN_18: no longer names the net of J13.18 (Pin_18)
- net PIN_2: no longer names the net of J13.2 (Pin_2)
- net PIN_20: no longer names the net of J13.20 (Pin_20)
- net PIN_4: no longer names the net of J13.4 (Pin_4)
- net PIN_6: no longer names the net of J13.6 (Pin_6)
- net PIN_8: no longer names the net of J13.8 (Pin_8)
- no-connect marks 15 -> 25
