File: spool/spool.kicad_sch (KiCad schematic)
At the start: 135 parts, among them J1 USB_B_Micro, J13 Conn_02x10_Counter_Clockwise, J14 Conn_01x07, J2 SWD, J3 Switch_1, J4 Switch_1, J5 Switch_1, J6 Switch_2, J7 Conn_01x02, J8 Conn_01x08, M1 Motor_DC, Q1 AO3400A, Q101 Q_NMOS_GSD, Q2 2N7002, SW1 USB_BOOT, SW2 RESET, SW3 SW_Push_DPDT, SW4 SW_Coded_SH-7010, SW5 SW_Push_DPDT, U1 TPS63070RNMR, U10 HT75xx-1-SOT89, U101 MMA8451QR1, U102 INA219AxDCN, U103 DY-ITR8402, U104 DY-ITR8402, U11 TPL0401B-10-Q1, U12 BS612, U14 PCF8563T, U3 AS5600-ASOT, U6 DRV8871DDA, U7 W25Q128JVS, U8 RP2040, U9 BS612, Y1 Crystal_GND24, Y2 Crystal

Commit message: Tidy up
Parts:
- BT1: LCSC C80909 -> (none); LCSC Part (none) -> C80909
- BZ1: LCSC C96256 -> (none); LCSC Part (none) -> C96256
- C1, C2: LCSC C45783 -> (none); LCSC Part (none) -> C45783
- C10, C4: LCSC C15525 -> (none); LCSC Part (none) -> C15525
- C101, C102, C104, C11, C12, C13, C14, C15, C16, C17, C18, C19, C22, C27, C28, C29, C33: LCSC C307331 -> (none); LCSC Part (none) -> C307331
- C103, C105, C3: LCSC C159814 -> (none); LCSC Part (none) -> C159814
- C20, C21, C25, C26, C30: LCSC C52923 -> (none); LCSC Part (none) -> C52923
- C23, C24: LCSC C1547 -> (none); LCSC Part (none) -> C1547
- C31, C32: LCSC C1555 -> (none); LCSC Part (none) -> C1555
- C34, C35: LCSC C3338 -> (none); LCSC Part (none) -> C3338
- C5, C6, C7, C8: LCSC C86295 -> (none); LCSC Part (none) -> C86295
- C9: LCSC C100072 -> (none); LCSC Part (none) -> C100072
- D1: LCSC C84256 -> (none); LCSC Part (none) -> C84256
- D10, D101, D11, D4, D5, D6, D7, D8, D9: LCSC C2128 -> (none); LCSC Part (none) -> C2128
- D2: LCSC C64898 -> (none); LCSC Part (none) -> C64898
- D3: LCSC C668989 -> (none); LCSC Part (none) -> C668989
- FB1: LCSC C76818 -> (none); LCSC Part (none) -> C76818
- J1: LCSC C145795 -> (none); LCSC Part (none) -> C145795
- J3, J4, J5, J6: LCSC C160388 -> (none); LCSC Part (none) -> C160388
- J7, R18: now not fitted
- J8: DigiKey Part (none) -> 455-S08B-XASK-1-ND; LCSC Part (none) -> C495695
- L1: LCSC C2042459 -> (none); LCSC Part (none) -> C2042459
- L101: footprint Connector_JST:JST_XA_B02B-XASK-1-A_1x02_P2.50mm_Vertical -> Connector_JST:JST_XA_B03B-XASK-1-A_1x03_P2.50mm_Vertical; LCSC C265077 -> (none); LCSC Part (none) -> C264992
- M1: LCSC C265077 -> (none); LCSC Part (none) -> C265077
- Q1: LCSC C20917 -> (none); LCSC Part (none) -> C20917
- Q101: LCSC C332302 -> (none); LCSC Part (none) -> C332302
- Q2: LCSC C8545 -> (none); LCSC Part (none) -> C8545
- R1: LCSC C319591 -> (none); LCSC Part (none) -> C319591
- R10, R101, R102, R12, R14, R4: LCSC C25741 -> (none); LCSC Part (none) -> C25741
- R103: value R_Shunt -> 100mΩ; LCSC Part (none) -> C25334
- R104, R105: LCSC C22808 -> (none); LCSC Part (none) -> C22808
- R16, R17: LCSC C25105 -> (none); LCSC Part (none) -> C25105
- R19, R24, R26, R30, R32: LCSC C11702 -> (none); LCSC Part (none) -> C11702
- R2, R20, R21, R22, R23, R25, R27, R28, R29, R6, R7: LCSC C25744 -> (none); LCSC Part (none) -> C25744
- R3: LCSC C723770 -> (none); LCSC Part (none) -> C723770
- R31: LCSC C25076 -> (none); LCSC Part (none) -> C25076
- R33: LCSC C17633 -> (none); LCSC Part (none) -> C17633
- RV1: LCSC C719176 -> (none); LCSC Part (none) -> C719176
- SW1, SW2: LCSC C318884 -> (none); LCSC Part (none) -> C318884
- SW3, SW5: LCSC C189615 -> (none); LCSC Part (none) -> C189615
- SW4: LCSC C440495 -> (none); LCSC Part (none) -> C440495
- U1: LCSC C109322 -> (none)
- U10: LCSC C14289 -> (none); LCSC Part (none) -> C14289
- U102: LCSC C87469 -> (none); LCSC Part (none) -> C87469
- U103, U104: LCSC C390039 -> (none); LCSC Part (none) -> C390039
- U11: LCSC C2666599 -> (none); LCSC Part (none) -> C2666599
- U14: LCSC C7440 -> (none); LCSC Part (none) -> C7440
- U6: LCSC C75864 -> (none); LCSC Part (none) -> C75864
- U7: LCSC C97521 -> (none); LCSC Part (none) -> C97521
- U8: LCSC C2040 -> (none)
- Y1: LCSC C9002 -> (none); LCSC Part (none) -> C9002
- Y2: LCSC C32346 -> (none); LCSC Part (none) -> C32346

Commit message: Tidy up
Parts:
- BT1: now left out of the parts list
Changed lines of the file:
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@@
 		(unit 1)
 		(exclude_from_sim no)
-		(in_bom yes)
+		(in_bom no)
 		(on_board yes)
 		(dnp no)

Commit message: Add Readme file
Other:
- note added: "Magnet rotary position sensor"
- note removed: "Magnet rotarty position sensor"
Changed lines of the file:
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@@
 		)
 	)
-	(text "Magnet rotarty \nposition sensor"
+	(text "Magnet rotary \nposition sensor"
 		(exclude_from_sim no)
 		(at 129.54 19.558 0)

Commit message: Add servo, more inputs and update board layout
Parts:
- removed C101, C102: 100n, Capacitor_SMD:C_0402_1005Metric, symbol Device:C_Small
- removed C103, C105: 2.2uF, Capacitor_SMD:C_0402_1005Metric, symbol Device:C_Small
- removed D1: LED, LED_SMD:LED_0805_2012Metric, symbol Device:LED
- removed J14: Conn_01x07, Connector_PinHeader_2.54mm:PinHeader_1x07_P2.54mm_Vertical, symbol Connector_Generic:Conn_01x07
- removed J3, J5: Switch_1, Connector_PinHeader_2.54mm:PinHeader_1x02_P2.54mm_Vertical, symbol Connector_Generic:Conn_01x02
- removed R24, R30: 1k, Resistor_SMD:R_0402_1005Metric, symbol Device:R
- removed R28, R29: 10k, Resistor_SMD:R_0402_1005Metric, symbol Device:R
- removed RV1: 10k, Potentiometer_SMD:Potentiometer_Bourns_TC33X_Vertical, symbol Device:R_Potentiometer
- removed SW3: SW_Push_DPDT, cacophony-library:SW-TH_K3-2235D-F1, symbol Switch:SW_Push_DPDT
- removed TP101: TestPoint, cacophony-library:TP_PAD, symbol cacophony-library:TestPoint
- removed U101: MMA8451QR1, cacophony-library:QFN-16_L3.0-W3.0-P0.50-TL_FXOS8700CQR1, symbol cacophony-library:MMA8451QR1
- removed U11: TPL0401B-10-Q1, Package_TO_SOT_SMD:Texas_R-PDSO-G6, symbol Potentiometer_Digital:TPL0401B-10-Q1
- removed U12, U9: BS612, cacophony-library:SENSORM-TH_BS612, symbol cacophony-library:BS612
- added C36, C46, C47, C48, C49, C50: 22uF, Capacitor_SMD:C_0603_1608Metric, symbol Device:C_Small
- added C37: 22nF, Capacitor_SMD:C_0402_1005Metric, symbol Device:C_Small
- added C38: 100nF, Capacitor_SMD:C_0402_1005Metric, symbol Device:C
- added C40: 100n, Capacitor_SMD:C_0402_1005Metric, symbol Device:C_Small
- added D17: D_Shockley, Diode_SMD:D_SMA, symbol Device:D_Shockley
- added H10, H9: MountingHole, cacophony-library:MountingHole_3.5mm_M3, symbol Mechanical:MountingHole
- added H11, H12, H13, H7, H8: MountingHole, cacophony-library:3.0mm_key_hole, symbol Mechanical:MountingHole
- added J3: Conn_01x03, Connector_JST:JST_SH_BM03B-SRSS-TB_1x03-1MP_P1.00mm_Vertical, symbol Connector_Generic_MountingPin:Conn_01x03_MountingPin
- added J5: Conn_01x03, Connector_PinHeader_2.54mm:PinHeader_1x03_P2.54mm_Vertical, symbol Connector_Generic:Conn_01x03
- added J9: Switch_2, Connector_JST:JST_SH_BM02B-SRSS-TB_1x02-1MP_P1.00mm_Vertical, symbol Connector_Generic_MountingPin:Conn_01x02_MountingPin
- added L2: 4.7uH, cacophony-library:IND-SMD_L7.0-W6.6, symbol Device:L
- added M2, M3: Servo, Connector_JST:JST_XA_B03B-XASK-1-A_1x03_P2.50mm_Vertical, symbol cacophony-library:Servo
- added R34, R35, R37, R38, R39, R40, R41, R43, R44: 1k, Resistor_SMD:R_0402_1005Metric, symbol Device:R
- added R42: 1k, Resistor_SMD:R_1206_3216Metric, symbol Device:R
- added TP2: TestPoint, TestPoint:TestPoint_Loop_D1.80mm_Drill1.0mm_Beaded, symbol cacophony-library:TestPoint
- added U2: PA_PIR, cacophony-library:PA_PIR, symbol cacophony-library:PA_PIR
- added U9: LMR14050S, Package_SO:TI_SO-PowerPAD-8, symbol cacophony-library:LMR14050S
- C27: value 100n -> 2.2uF; LCSC Part C307331 -> C159814
- C28, C29: value 100n -> 22uF; footprint Capacitor_SMD:C_0402_1005Metric -> Capacitor_SMD:C_0805_2012Metric; LCSC (none) -> C45783; LCSC Part C307331 -> (none)
- J2: footprint Connector_PinHeader_2.54mm:PinHeader_1x03_P2.54mm_Vertical -> Connector_PinHeader_1.00mm:PinHeader_1x03_P1.00mm_Vertical
- J4, J6: footprint cacophony-library:JST_SH_BM02B-SRSS-TB_1x02-1MP_P1.00mm_Vertical -> Connector_JST:JST_SH_BM02B-SRSS-TB_1x02-1MP_P1.00mm_Vertical; symbol Connector_Generic:Conn_01x02 -> Connector_Generic_MountingPin:Conn_01x02_MountingPin
- L101: footprint Connector_JST:JST_XA_B03B-XASK-1-A_1x03_P2.50mm_Vertical -> cacophony-library:JST_XA_B03B_2_Pin
- R22: value 10k -> 47k; LCSC (none) -> C25792; LCSC Part C25744 -> (none)
- R23: LCSC (none) -> C25744; LCSC Part C25744 -> (none)
- R25: value 10k -> 100k; LCSC (none) -> C25741; LCSC Part C25744 -> (none)
- R26: value 1k -> 560; footprint Resistor_SMD:R_0402_1005Metric -> Resistor_SMD:R_0603_1608Metric; LCSC (none) -> C23204; LCSC Part C11702 -> (none)
- R27: value 10k -> 680; footprint Resistor_SMD:R_0402_1005Metric -> Resistor_SMD:R_0603_1608Metric; LCSC (none) -> C23228; LCSC Part C25744 -> (none)
- SW1, SW2: footprint Button_Switch_SMD:SW_SPST_SKQG_WithStem -> cacophony-library:SW_SPST_SKQG_WithStem
Connections:
- net GPIO_21 is gone; now on net RELEASE: U8.32 (GPIO21)
- net PIR_2 is gone; now on net H_IN1: U8.15 (GPIO12)
- net PIR_SENS_POT_PROG is gone; now on an unnamed net: R27.1
- net +12V: now also C27.1, C28.1, C29.1, J13.7 (Pin_7), J13.9 (Pin_9), R42.2, U9.2 (VIN); no longer J13.1 (Pin_1), J13.3 (Pin_3)
- net +3V3: now also J13.1 (Pin_1), J13.3 (Pin_3); no longer J13.7 (Pin_7), J13.9 (Pin_9)
- net +3V3_Lin: now also C40.1, U2.3 (VDD); no longer C27.1, C28.1, C29.1, R22.1, R23.2, R27.2
- net GND: now also J1.SH (Shield), R22.2, R27.2, C36.2, C37.2, C40.2, C46.2, C47.2, C48.2, C49.2, C50.2, D17.2 (A), J3.2 (Pin_2), J9.1 (Pin_1), M2.1 (GND), M3.1 (GND), U2.1 (GND), U9.7 (GND), U9.9 (PGND); no longer J1.6 (Shield)
- net H_IN1: now also D5.2 (A), R10.1; no longer U8.12 (GPIO9)
- net H_IN2: now also D4.2 (A), R12.1, U8.16 (GPIO13); no longer U8.13 (GPIO10)
- net PHOTO_HOME_OUT: now also U8.14 (GPIO11); no longer U8.18 (GPIO15)
- net PHOTO_RESET_OUT: now also U8.13 (GPIO10); no longer U8.17 (GPIO14)
- net RELEASE: no longer U8.29 (GPIO18)
- net RP2040_RX_IN: now also U8.28 (GPIO17); no longer U8.41 (GPIO29_ADC3)
- net RP2040_TX_IN: now also R44.2; no longer U8.40 (GPIO28_ADC2)
- net RP2040_TX_OUT: now also R43.2; no longer U8.36 (GPIO24)
- net RTC_BAT_SENSE: now also TP2.1; no longer U8.38 (GPIO26_ADC0)
- net R_ENC_1: now also U8.11 (GPIO8); no longer U8.6 (GPIO4)
- net R_ENC_2: now also U8.5 (GPIO3); no longer U8.7 (GPIO5)
- net R_ENC_4: now also U8.9 (GPIO7); no longer U8.5 (GPIO3)
- net R_ENC_8: now also U8.6 (GPIO4); no longer U8.8 (GPIO6)
- net SCL: now also J13.6 (Pin_6), U8.18 (GPIO15); no longer J13.8 (Pin_8), U8.28 (GPIO17)
- net SDA: now also J13.8 (Pin_8), U8.17 (GPIO14); no longer J13.6 (Pin_6), U8.27 (GPIO16)
- net SWITCH_1: now also R38.2; no longer U8.9 (GPIO7)
- net SWITCH_2: now also R40.2; no longer U8.11 (GPIO8)
- net at D10.1 (K), D9.1 (K), U6.3 (IN1): no longer D5.2 (A), R10.1
- net GPIO_12: now reaches J13.4 (Pin_4)
- net GPIO_12: now also U8.35 (GPIO23)
- net at D7.1 (K), D8.1 (K), U6.2 (IN2): no longer D4.2 (A), R12.1
- net EN_PHOTO_PHY: now reaches D6.2 (A)
- net EN_PHOTO_PHY: now also U8.12 (GPIO9); no longer U8.14 (GPIO11)
- net EN_6V: now reaches R25.2
- net EN_6V: now also U8.29 (GPIO18), U9.3 (EN)
- net Accel INT1 renamed SERVO_1_PHY
- net SERVO_1_PHY: now also R35.1
- net GPIO_20 renamed SERVO_2_PHY
- net SERVO_2_PHY: now also R34.1
- net GPIO_27 renamed ADC1
- net ADC1: now also J5.1 (Pin_1)
- net GPIO_34 renamed PIR_EX_PHY
- net PIR_EX_PHY: now also R41.1
- net LED_1_PHY renamed SW_1_PHY
- net SW_1_PHY: now also R38.1
- net PIR_1: no longer names the net of R26.1
- net PIR_1: now also R23.2, U9.5 (FB); no longer U8.16 (GPIO13)
- net PIR_SENS_POT_MANUAL renamed +6V
- net +6V: now also C36.1, C46.1, C47.1, C48.1, C49.1, C50.1, L2.2, M2.2 (+Ve), M3.2 (+Ve)
- net ~{RTC_INT}: no longer names the net of U14.3 (~{INT})
- net ~{RTC_INT}: no longer U8.35 (GPIO23)
- new net: C37.1, U9.6 (SS)
- new net: C38.2, U9.1 (Boot)
- new net: R22.1, U9.4 (RT/SYNC)
- new net ADC2: J5.2 (Pin_2), U8.40 (GPIO28_ADC2)
- new net ADC3: J5.3 (Pin_3), U8.41 (GPIO29_ADC3)
- new net APIR: R37.2, U2.2 (OUT)
- new net APIR_PHY: R37.1, U8.38 (GPIO26_ADC0)
- new net EX_PIR_POWER: J3.1 (Pin_1), R42.1
- new net PIR_EX: J3.3 (Pin_3), R41.2
- new net RP2040_TX_IN_PHY: R44.1, U8.27 (GPIO16)
- new net RP2040_TX_OUT_PHY: R43.1, U8.36 (GPIO24)
- new net SERVO_1: M3.3 (SIG), R35.2
- new net SERVO_2: M2.3 (SIG), R34.2
- new net SPOOL_REED: J9.2 (Pin_2), R39.2
- new net SPOOL_REED_PHY: R39.1, U8.8 (GPIO6)
- new net SW_2_PHY: R40.1, U8.7 (GPIO5)
- new net SW_6V: C38.1, D17.1 (K), L2.1, U9.8 (SW)
- no-connect marks 29 -> 22
Other:
- note removed: "Accelerometer"
- note removed: "PIRs"
- note removed: "Sensitivity for PIRs"
- moved on the sheet: C1, C104, C2, C25, C26, C3, C33, C34, C35, C4, C5, C6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

Commit message: Update to use new PIR and added servo outputs
Parts:
- added C39: 100n, Capacitor_SMD:C_0402_1005Metric, symbol Device:C
- added J1901: TC2030, cacophony-library:Tag-Connect_TC2030-IDC-NL_2x03_P1.27mm_Vertical, symbol Connector:TC2030
- added R115: 100k, Resistor_SMD:R_0402_1005Metric, symbol Device:R
- added U106: M24C02-WMN, Package_SO:SOIC-8_3.9x4.9mm_P1.27mm, symbol Memory_EEPROM:M24C02-WMN
- added U4: (no value), cacophony-library:JLCPCB_QR_8mm, symbol cacophony-library:JLCPCB_QR_CODE
- C28, C29: LCSC C45783 -> (none); LCSC Part (none) -> C45783
- C37: LCSC C1532 -> (none); LCSC Part (none) -> C1532
- C38: LCSC C1525 -> (none); LCSC Part (none) -> C1525
- D17: LCSC C22452 -> (none); LCSC Part (none) -> C22452
- J3: LCSC Part (none) -> C160389
- J5, U2: now left out of the parts list
- L2: LCSC C408447 -> (none); LCSC Part (none) -> C408447
- M2, M3: LCSC C264992 -> (none); LCSC Part (none) -> C264992
- R22: LCSC C25792 -> (none); LCSC Part (none) -> C25792
- R23: LCSC C25744 -> (none); LCSC Part (none) -> C25744
- R25: LCSC C25741 -> (none); LCSC Part (none) -> C25741
- R26: LCSC C23204 -> (none); LCSC Part (none) -> C23204
- R27: LCSC C23228 -> (none); LCSC Part (none) -> C23228
- U9: LCSC C155484 -> (none); LCSC Part (none) -> C155484
Connections:
- net +3V3: now also C39.2, R115.2, U106.8 (VCC)
- net GND: now also C39.1, J1901.5, U106.4 (VSS)
- net PHOTO_HOME_OUT: now also U8.13 (GPIO10); no longer U8.14 (GPIO11)
- net PHOTO_RESET_OUT: now also U8.14 (GPIO11); no longer U8.13 (GPIO10)
- net SCL: now also J1901.4, U106.6 (SCL)
- net SDA: now also J1901.2, U106.5 (SDA)
- new net EEPROM_~{WC}: J1901.1, R115.1, U106.7 (~{WC})
- no-connect marks 22 -> 27
Other:
- note added: "EEPROM 2K"
- note added: "I2C Address 0x50"

Commit message: Added kicad-library as submodule and simplify schematic
Parts:
- removed D3: D, Diode_SMD:D_SOD-523, symbol Device:D
- removed J7: Conn_01x02, Connector_PinHeader_2.00mm:PinHeader_1x02_P2.00mm_Vertical, symbol Connector_Generic:Conn_01x02
- removed JP1: SolderJumper_2_Bridged, Jumper:SolderJumper-2_P1.3mm_Bridged_RoundedPad1.0x1.5mm, symbol Jumper:SolderJumper_2_Bridged
- removed R42: 1k, Resistor_SMD:R_1206_3216Metric, symbol Device:R
- added R45, R46, R47, R48: 1k, Resistor_SMD:R_0402_1005Metric, symbol Device:R
- C1, C2, C28, C29: value 22uF -> 22uF 25V
- C104, C11, C12, C13, C14, C15, C16, C17, C18, C19, C22, C33, C39, C40: value 100n -> 100nF
- C38: LCSC Part C1525 -> C307331
- C9: LCSC Part C100072 -> C307331
- D10, D101, D11, D4, D5, D6, D7, D8, D9: footprint Diode_SMD:D_SOD-323_HandSoldering -> Diode_SMD:D_SOD-323
- D2: footprint Diode_SMD:D_SOD-123F -> Diode_SMD:D_SOD-323; LCSC Part C64898 -> C2128
Connections:
- net RTC_BAT_SENSE is gone; now on net RTC_BAT: TP2.1
- net +12V: now also R47.2, R48.2
- net EX_PIR_POWER: now also R45.1, R46.1
- net RTC_BAT: now also BT1.1 (+)
- new net: R45.2, R46.2, R47.1, R48.1
Other:
- note added: "Using 4 1k 0402 resistors to increase the wattage so we don't need a different component."
- moved on the sheet: C30, TP2
