File: spool-plugs/spool-plugs.kicad_sch (KiCad schematic)
At the start: 7 parts, among them J2 JCON_M16_04Pin, J4 Conn_01x08, J5 JCON_M16_2+4Pin, J6 JCON_M16_2+4Pin

Commit message: Move files
Parts:
- D201: renamed from D1; LCSC C22452 -> (none); LCSC Part (none) -> C22452
- D202: renamed from D3; LCSC C22452 -> (none); LCSC Part (none) -> C22452
- D203: renamed from D2; LCSC C22452 -> (none); LCSC Part (none) -> C22452
- J202: renamed from J4; LCSC Part (none) -> C495695
- renumbered J2 to J201, J5 to J203, J6 to J204
Connections:
- net RP2040_RX_IN: now also J202.2 (Pin_2); no longer J202.7 (Pin_7)
- net RP2040_RX_OUT: now also J202.5 (Pin_5); no longer J202.4 (Pin_4)
- net RP2040_TX_IN: now also J202.1 (Pin_1); no longer J202.8 (Pin_8)
- net RP2040_TX_OUT: now also J202.4 (Pin_4); no longer J202.5 (Pin_5)
- net VCC: now also J202.7 (Pin_7), J202.8 (Pin_8); no longer J202.1 (Pin_1), J202.2 (Pin_2)
Other:
- moved on the sheet: J202
Changed lines of the file:
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@@
 		(on_board yes)
 		(dnp no)
-		(property "Reference" "D3"
+		(property "Reference" "D202"
 			(at 175.26 66.04 0)
 			(effects
@@
 			)
 		)
-		(property "LCSC" "C22452"
-			(at 175.26 60.96 0)
-			(effects
-				(font
-					(size 1.27 1.27)
-				)
-				(hide yes)
-			)
-		)
 		(property "Digikey" "641-SS54-HFCT-ND"
 			(at 175.26 60.96 0)
@@
 			)
 		)
+		(property "LCSC Part" "C22452"
+			(at 175.26 60.96 0)
+			(effects
+				(font
+					(size 1.27 1.27)
+				)
+				(hide yes)
+			)
+		)
+		(property "LCSC" ""
+			(at 175.26 60.96 0)
+			(effects
+				(font
+					(size 1.27 1.27)
+				)
+				(hide yes)
+			)
+		)
 		(pin "1"
 		)
@@
 			(project "trap-plugs"
 				(path "/2aa3d595-b075-467f-ac50-47a0458f5456"
-					(reference "D3")
+					(reference "D202")
 					(unit 1)
 				)
@@
 		(dnp no)
 		(fields_autoplaced yes)
-		(property "Reference" "D1"
+		(property "Reference" "D201"
 			(at 85.09 35.56 0)
 			(effects
@@
 			)
 		)
-		(property "LCSC" "C22452"
-			(at 85.09 41.91 0)
-			(effects
-				(font
-					(size 1.27 1.27)
-				)
-				(hide yes)
-			)
-		)
 		(property "Digikey" "641-SS54-HFCT-ND"
 			(at 85.09 41.91 0)
@@
 			)
 		)
+		(property "LCSC Part" "C22452"
+			(at 85.09 41.91 0)
+			(effects
+				(font
+					(size 1.27 1.27)
+				)
+				(hide yes)
+			)
+		)
+		(property "LCSC" ""
+			(at 85.09 41.91 0)
+			(effects
+				(font
+					(size 1.27 1.27)
+				)
+				(hide yes)
+			)
+		)
 		(pin "1"
 		)
@@
 			(project "trap-plugs"
 				(path "/2aa3d595-b075-467f-ac50-47a0458f5456"
-					(reference "D1")
+					(reference "D201")
 					(unit 1)
 				)
@@
 		(dnp no)
 		(fields_autoplaced yes)
-		(property "Reference" "#PWR04"
+		(property "Reference" "#PWR0207"
 			(at 228.6 68.58 0)
 			(effects
@@
 			(project "trap-plugs"
 				(path "/2aa3d595-b075-467f-ac50-47a0458f5456"
-					(reference "#PWR04")
+					(reference "#PWR0207")
 					(unit 1)
 				)
@@
 		(dnp no)
 		(fields_autoplaced yes)
-		(property "Reference" "J6"
+		(property "Reference" "J204"
 			(at 237.49 45.72 0)
 			(effects
@@
 			)
 		)
+		(property "LCSC" ""
+			(at 237.49 57.15 0)
+			(effects
+				(font
+					(size 1.27 1.27)
+				)
+				(hide yes)
+			)
+		)
 		(pin "1"
 		)
@@
 			(project "trap-plugs"
 				(path "/2aa3d595-b075-467f-ac50-47a0458f5456"
-					(reference "J6")
+					(reference "J204")
 					(unit 1)
 				)
@@
 		(dnp no)
 		(fields_autoplaced yes)
-		(property "Reference" "#PWR07"
+		(property "Reference" "#PWR0206"
 			(at 185.42 63.5 0)
 			(effects
@@
 			(project "trap-plugs"
 				(path "/2aa3d595-b075-467f-ac50-47a0458f5456"
-					(reference "#PWR07")
+					(reference "#PWR0206")
 					(unit 1)
 				)
@@
 		(dnp no)
 		(fields_autoplaced yes)
-		(property "Reference" "#PWR02"
+		(property "Reference" "#PWR0203"
 			(at 106.68 140.97 0)
 			(effects
@@
 			(project "trap-plugs"
 				(path "/2aa3d595-b075-467f-ac50-47a0458f5456"
-					(reference "#PWR02")
+					(reference "#PWR0203")
 					(unit 1)
 				)
@@
 		(dnp no)
 		(fields_autoplaced yes)
-		(property "Reference" "#PWR03"
+		(property "Reference" "#PWR0204"
 			(at 143.51 68.58 0)
 			(effects
@@
 			(project "trap-plugs"
 				(path "/2aa3d595-b075-467f-ac50-47a0458f5456"
-					(reference "#PWR03")
+					(reference "#PWR0204")
 					(unit 1)
 				)
@@
 	(symbol
 		(lib_id "Connector_Generic:Conn_01x08")
-		(at 100.33 124.46 180)
+		(at 100.33 121.92 0)
+		(mirror y)
 		(unit 1)
 		(exclude_from_sim no)
@@
 		(on_board yes)
 		(dnp no)
-		(fields_autoplaced yes)
-		(property "Reference" "J4"
-			(at 100.33 107.95 0)
+		(property "Reference" "J202"
+			(at 100.33 138.43 0)
 			(effects
 				(font
@@
 		)
 		(property "Value" "Conn_01x08"
-			(at 100.33 110.49 0)
+			(at 100.33 135.89 0)
 			(effects
 				(font
@@
 		)
 		(property "Footprint" "Connector_JST:JST_XA_S08B-XASK-1_1x08_P2.50mm_Horizontal"
-			(at 100.33 124.46 0)
+			(at 100.33 121.92 0)
 			(effects
 				(font
@@
 		)
 		(property "Datasheet" "~"
-			(at 100.33 124.46 0)
+			(at 100.33 121.92 0)
 			(effects
 				(font
@@
 		)
 		(property "Description" "Generic connector, single row, 01x08, script generated (kicad-library-utils/schlib/autogen/connector/)"
-			(at 100.33 124.46 0)
+			(at 100.33 121.92 0)
 			(effects
 				(font
@@
 		)
 		(property "Digikey" "641-SS54-HFCT-ND"
-			(at 100.33 124.46 0)
+			(at 100.33 121.92 0)
+			(effects
+				(font
+					(size 1.27 1.27)
+				)
+				(hide yes)
+			)
+		)
+		(property "LCSC Part" "C495695"
+			(at 100.33 121.92 0)
+			(effects
+				(font
+					(size 1.27 1.27)
+				)
+				(hide yes)
+			)
+		)
+		(property "LCSC" ""
+			(at 100.33 121.92 0)
 			(effects
 				(font
@@
 			(project "trap-plugs"
 				(path "/2aa3d595-b075-467f-ac50-47a0458f5456"
-					(reference "J4")
+					(reference "J202")
 					(unit 1)
 				)
@@
 		(dnp no)
 		(fields_autoplaced yes)
-		(property "Reference" "#FLG03"
+		(property "Reference" "#FLG0201"
 			(at 69.85 57.785 0)
 			(effects
@@
 			(project "trap-plugs"
 				(path "/2aa3d595-b075-467f-ac50-47a0458f5456"
-					(reference "#FLG03")
+					(reference "#FLG0201")
 					(unit 1)
 				)
@@
 		(dnp no)
 		(fields_autoplaced yes)
-		(property "Reference" "#PWR01"
+		(property "Reference" "#PWR0208"
 			(at 267.97 62.23 0)
 			(effects
@@
 			(project "trap-plugs"
 				(path "/2aa3d595-b075-467f-ac50-47a0458f5456"
-					(reference "#PWR01")
+					(reference "#PWR0208")
 					(unit 1)
 				)
@@
 		(dnp no)
 		(fields_autoplaced yes)
-		(property "Reference" "#FLG01"
+		(property "Reference" "#FLG0202"
 			(at 138.43 128.905 0)
 			(effects
@@
 			(project "trap-plugs"
 				(path "/2aa3d595-b075-467f-ac50-47a0458f5456"
-					(reference "#FLG01")
+					(reference "#FLG0202")
 					(unit 1)
 				)
@@
 		(on_board yes)
 		(dnp no)
-		(property "Reference" "D2"
+		(property "Reference" "D203"
 			(at 255.27 66.04 0)
 			(effects
@@
 			)
 		)
-		(property "LCSC" "C22452"
-			(at 255.27 60.96 0)
-			(effects
-				(font
-					(size 1.27 1.27)
-				)
-				(hide yes)
-			)
-		)
 		(property "Digikey" "641-SS54-HFCT-ND"
 			(at 255.27 60.96 0)
@@
 			)
 		)
+		(property "LCSC Part" "C22452"
+			(at 255.27 60.96 0)
+			(effects
+				(font
+					(size 1.27 1.27)
+				)
+				(hide yes)
+			)
+		)
+		(property "LCSC" ""
+			(at 255.27 60.96 0)
+			(effects
+				(font
+					(size 1.27 1.27)
+				)
+				(hide yes)
+			)
+		)
 		(pin "1"
 		)
@@
 			(project "trap-plugs"
 				(path "/2aa3d595-b075-467f-ac50-47a0458f5456"
-					(reference "D2")
+					(reference "D203")
 					(unit 1)
 				)
@@
 		(on_board yes)
 		(dnp no)
-		(property "Reference" "J2"
+		(property "Reference" "J201"
 			(at 59.69 39.37 0)
 			(effects
@@
 			)
 		)
+		(property "LCSC" ""
+			(at 59.69 48.26 0)
+			(effects
+				(font
+					(size 1.27 1.27)
+				)
+				(hide yes)
+			)
+		)
 		(pin "1"
 		)
@@
 			(project "trap-plugs"
 				(path "/2aa3d595-b075-467f-ac50-47a0458f5456"
-					(reference "J2")
+					(reference "J201")
 					(unit 1)
 				)
@@
 		(dnp no)
 		(fields_autoplaced yes)
-		(property "Reference" "#PWR06"
+		(property "Reference" "#PWR0201"
 			(at 73.66 62.23 0)
 			(effects
@@
 			(project "trap-plugs"
 				(path "/2aa3d595-b075-467f-ac50-47a0458f5456"
-					(reference "#PWR06")
+					(reference "#PWR0201")
 					(unit 1)
 				)
@@
 		(dnp no)
 		(fields_autoplaced yes)
-		(property "Reference" "J5"
+		(property "Reference" "J203"
 			(at 152.4 45.72 0)
 			(effects
@@
 			)
 		)
+		(property "LCSC" ""
+			(at 152.4 57.15 0)
+			(effects
+				(font
+					(size 1.27 1.27)
+				)
+				(hide yes)
+			)
+		)
 		(pin "1"
 		)
@@
 			(project "trap-plugs"
 				(path "/2aa3d595-b075-467f-ac50-47a0458f5456"
-					(reference "J5")
+					(reference "J203")
 					(unit 1)
 				)
@@
 		(dnp no)
 		(fields_autoplaced yes)
-		(property "Reference" "#PWR08"
+		(property "Reference" "#PWR0205"
 			(at 152.4 134.62 0)
 			(effects
@@
 			(project "trap-plugs"
 				(path "/2aa3d595-b075-467f-ac50-47a0458f5456"
-					(reference "#PWR08")
+					(reference "#PWR0205")
 					(unit 1)
 				)
@@
 		(dnp no)
 		(fields_autoplaced yes)
-		(property "Reference" "#PWR05"
+		(property "Reference" "#PWR0202"
 			(at 95.25 44.45 0)
 			(effects
@@
 			(project "trap-plugs"
 				(path "/2aa3d595-b075-467f-ac50-47a0458f5456"
-					(reference "#PWR05")
-					(unit 1)
-				)
+					(reference "#PWR0202")
+					(unit 1)
+				)
