File: spool-plugs/spool-plugs.kicad_sch (KiCad schematic)
At the start: 7 parts, among them J201 JCON_M16_04Pin, J202 Conn_01x08, J203 JCON_M16_2+4Pin, J204 JCON_M16_2+4Pin

Commit message: Adding STM32 version
Parts:
- removed D203: D_Shockley, Diode_SMD:D_SMA_Handsoldering, symbol Device:D_Shockley
- removed J202: Conn_01x08, Connector_JST:JST_XA_S08B-XASK-1_1x08_P2.50mm_Horizontal, symbol Connector_Generic:Conn_01x08
- removed J204: JCON_M16_2+4Pin, cacophony-library:jcon-2+4pin-m16, symbol cacophony-library:JCON_M16_2+4Pin
- added D204: D_Zener, Diode_SMD:Littelfuse_PolyZen-LS, symbol Device:D_Zener
- added H201, H202, H203: MountingHole, cacophony-library:3.0mm_key_hole, symbol Mechanical:MountingHole
- added J205: JCON_M16_8Pin, cacophony-library:jcon-8pin-m16, symbol cacophony-library:JCON_M16_8Pin
- added J209: Conn_02x10_Odd_Even, cacophony-library:spool_pcb-pcb_connector, symbol Connector_Generic:Conn_02x10_Odd_Even
- added R201: 4.7M, Resistor_SMD:R_0805_2012Metric, symbol Device:R
- added R202, R203: 1M, Resistor_SMD:R_0805_2012Metric, symbol Device:R
Connections:
- net GND: now also J205.7, J209.17 (Pin_17), J209.18 (Pin_18), J209.5 (Pin_5), J209.6 (Pin_6), R202.2, R203.2
- net RP2040_RX_IN: now also J209.19 (Pin_19)
- net RP2040_TX_IN: now also J209.20 (Pin_20)
- net VCC: now also J209.1 (Pin_1), J209.4 (Pin_4)
- net +Batt renamed BAT_SENSE
- net BAT_SENSE: now also D204.1 (K), R201.1
- new net: D204.2 (A), R203.1
- new net BAT_DIV: J209.15 (Pin_15), R201.2, R202.1
- new net EX_PIR_POWER: J205.8, J209.16 (Pin_16)
- new net PIR_EX: J205.1, J209.12 (Pin_12)
- new net REED_SW_1: J205.3, J209.10 (Pin_10)
- new net REED_SW_2: J205.2, J209.9 (Pin_9)
- new net SERVO_SIG_1: J205.4, J209.7 (Pin_7)
- new net SERVO_SIG_2: J205.5, J209.8 (Pin_8)
- new net SPOOL_POWER: J205.6, J209.2 (Pin_2), J209.3 (Pin_3)
- no-connect marks 2 -> 4
Other:
- moved on the sheet: D201, D202, J201, J203
