File: spool-plugs/spool-plugs.kicad_pcb (KiCad board)
At the start: 4 copper layers, 58 x 29 mm, 7 parts, among them J201 JCON_M16_04Pin, J202 Conn_01x08, J203 JCON_M16_2+4Pin, J204 JCON_M16_2+4Pin

Commit message: Update to use new PIR and added servo outputs
Other:
- board text added: "Spool Plugs ${TAG} ${HASH}"
- board text added: "VIN"
- board text removed: "Spool Plugs ${TAG}"
