File: spool-plugs/spool-plugs.kicad_pcb (KiCad board)
At the start: 4 copper layers, 58 x 29 mm, 7 parts, among them J201 JCON_M16_04Pin, J202 Conn_01x08, J203 JCON_M16_2+4Pin, J204 JCON_M16_2+4Pin

Commit message: Adding STM32 version
Parts:
- removed D203: D_Shockley, Diode_SMD:D_SMA_Handsoldering
- removed J202: Conn_01x08, Connector_JST:JST_XA_S08B-XASK-1_1x08_P2.50mm_Horizontal
- removed J204: JCON_M16_2+4Pin, cacophony-library:jcon-2+4pin-m16
- added D204: D_Zener, Diode_SMD:Littelfuse_PolyZen-LS, F.Cu at (-0.27, -2.44)
- added H201: MountingHole, cacophony-library:3.0mm_key_hole, F.Cu at (2.00, 12.0)
- added H202: MountingHole, cacophony-library:3.0mm_key_hole, F.Cu at (25.0, -14.0)
- added H203: MountingHole, cacophony-library:3.0mm_key_hole, F.Cu at (-25.0, -14.0)
- added J205: JCON_M16_8Pin, cacophony-library:jcon-8pin-m16, F.Cu at (-23.0, 0.00)
- added J209: Conn_02x10_Odd_Even, cacophony-library:spool_pcb-pcb_connector, F.Cu at (-4.49, 12.1)
- added R201: 4.7M, Resistor_SMD:R_0805_2012Metric, F.Cu at (3.21, -3.06)
- added R202: 1M, Resistor_SMD:R_0805_2012Metric, F.Cu at (3.18, 0.43)
- added R203: 1M, Resistor_SMD:R_0805_2012Metric, F.Cu at (1.07, 2.03)
- moved D202 174.2 mm to (12.3, -1.77)
- moved J203 172.4 mm to (23.0, 0.00)
- moved J201 172.3 mm to (0.01, -11.3)
- moved D201 167.2 mm to (-6.62, -2.90), turned to 90 degrees
Connections:
- J201 pad 4: /+Batt -> /BAT_SENSE
Routing:
- net SPEAKER_-: track 59.2 -> 0.00 mm, vias 2 -> 0
- net SPEAKER_+: track 56.5 -> 0.00 mm, vias 1 -> 0
- net EX_PIR_POWER: track 0.00 -> 24.0 mm
- net RP2040_RX_OUT: track 23.5 -> 0.00 mm
- net RP2040_TX_OUT: track 21.0 -> 0.00 mm
- net BAT_DIV: track 0.00 -> 20.2 mm
- net SPOOL_POWER: track 0.00 -> 19.9 mm
- net PIR_EX: track 0.00 -> 19.2 mm
- net VCC: track 17.0 -> 0.00 mm, vias 9 -> 0
- net SERVO_SIG_2: track 0.00 -> 16.4 mm
- net /BAT_SENSE: track 0.00 -> 14.5 mm
- net REED_SW_1: track 0.00 -> 13.8 mm
- net REED_SW_2: track 0.00 -> 12.2 mm
- net SERVO_SIG_1: track 0.00 -> 11.5 mm
- net /VOUT_PHY: track 6.46 -> 0.00 mm
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Other:
- board size 58 x 29 mm -> 58 x 35.7 mm
- board text removed: "GND"
- board text removed: "In"
- board text removed: "Out"
- board text removed: "Power"
- board text removed: "RX_IN"
- board text removed: "RX_OUT"
- board text removed: "TX_IN"
- board text removed: "TX_OUT"
- board text removed: "VCC"
- board text removed: "VIN"
